File: time_output.sch (KiCad schematic (older format))
At the start: 3 parts, among them P1 BNC, U12 74LVC14

Commit message: R2 PCB rotary switches closer to middle of board
Parts:
- U12: Distributor (none) -> Mouser; Distributor PN (none) -> 595-SN74LVC14ADR; Manufacturer (none) -> TI; Manufacturer PN (none) -> SN74LVC14ADR; URL (none) -> http://www.mouser.com/Search/ProductDetail.aspx?R=SN74LVC14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; Unit Price (none) -> 0.40
Changed lines of the file:
@@
 encoding utf-8
 Sheet 4 6
-Title ""
+Title "calbox time output"
 Date ""
 Rev ""
@@
 Connection ~ 6100 1300
 $Comp
-L GND #PWR62
+L GND #PWR048
 U 1 1 58C45355
 P 7100 1500
-F 0 "#PWR62" H 7100 1250 50  0001 C CNN
+F 0 "#PWR048" H 7100 1250 50  0001 C CNN
 F 1 "GND" H 7100 1350 50  0000 C CNN
 F 2 "" H 7100 1500 50  0000 C CNN
@@
 F 1 "74LVC14" H 4550 1200 50  0000 C CNN
 F 2 "SMD_Packages:SOIC-14_N" H 4350 1300 50  0001 C CNN
-F 3 "" H 4350 1300 50  0000 C CNN
+F 3 "http://www.ti.com/lit/ds/symlink/sn74lvc14a.pdf" H 4350 1300 50  0001 C CNN
+F 4 "TI" H 4350 1300 60  0001 C CNN "Manufacturer"
+F 5 "SN74LVC14ADR" H 4350 1300 60  0001 C CNN "Manufacturer PN"
+F 6 "Mouser" H 4350 1300 60  0001 C CNN "Distributor"
+F 7 "595-SN74LVC14ADR" H 4350 1300 60  0001 C CNN "Distributor PN"
+F 8 "http://www.mouser.com/Search/ProductDetail.aspx?R=SN74LVC14ADRvirtualkey59500000virtualkey595-SN74LVC14ADR" H 4350 1300 60  0001 C CNN "URL"
+F 9 "0.40" H 4350 1300 60  0001 C CNN "Unit Price"
 	1    4350 1300
 	1    0    0    -1
 $EndComp
 $Comp
-L 74LVC14 U12
-U 2 1 58C46AA2
-P 5450 1300
-F 0 "U12" H 5600 1400 50  0000 C CNN
-F 1 "74LVC14" H 5650 1200 50  0000 C CNN
-F 2 "SMD_Packages:SOIC-14_N" H 5450 1300 50  0001 C CNN
-F 3 "" H 5450 1300 50  0000 C CNN
-	2    5450 1300
-	1    0    0    -1
-$EndComp
-$Comp
-L GND #PWR51
+L GND #PWR049
 U 1 1 58C46B80
 P 4300 1500
-F 0 "#PWR51" H 4300 1250 50  0001 C CNN
+F 0 "#PWR049" H 4300 1250 50  0001 C CNN
 F 1 "GND" H 4300 1350 50  0000 C CNN
 F 2 "" H 4300 1500 50  0000 C CNN
@@
 $EndComp
 $Comp
-L GND #PWR53
+L GND #PWR050
 U 1 1 58C46BA0
 P 5400 1500
-F 0 "#PWR53" H 5400 1250 50  0001 C CNN
+F 0 "#PWR050" H 5400 1250 50  0001 C CNN
 F 1 "GND" H 5400 1350 50  0000 C CNN
 F 2 "" H 5400 1500 50  0000 C CNN
@@
 $EndComp
 $Comp
-L 74LVC14 U12
-U 3 1 58C46C7A
-P 5450 2100
-F 0 "U12" H 5600 2200 50  0000 C CNN
-F 1 "74LVC14" H 5650 2000 50  0000 C CNN
-F 2 "SMD_Packages:SOIC-14_N" H 5450 2100 50  0001 C CNN
-F 3 "" H 5450 2100 50  0000 C CNN
-	3    5450 2100
-	1    0    0    -1
-$EndComp
-$Comp
-L GND #PWR55
+L GND #PWR051
 U 1 1 58C470F0
 P 5400 2300
-F 0 "#PWR55" H 5400 2050 50  0001 C CNN
+F 0 "#PWR051" H 5400 2050 50  0001 C CNN
 F 1 "GND" H 5400 2150 50  0000 C CNN
 F 2 "" H 5400 2300 50  0000 C CNN
@@
 $EndComp
 $Comp
-L 74LVC14 U12
-U 4 1 58C4710C
-P 5450 2900
-F 0 "U12" H 5600 3000 50  0000 C CNN
-F 1 "74LVC14" H 5650 2800 50  0000 C CNN
-F 2 "SMD_Packages:SOIC-14_N" H 5450 2900 50  0001 C CNN
-F 3 "" H 5450 2900 50  0000 C CNN
-	4    5450 2900
-	1    0    0    -1
-$EndComp
-$Comp
-L GND #PWR57
+L GND #PWR052
 U 1 1 58C47146
 P 5400 3100
-F 0 "#PWR57" H 5400 2850 50  0001 C CNN
+F 0 "#PWR052" H 5400 2850 50  0001 C CNN
 F 1 "GND" H 5400 2950 50  0000 C CNN
 F 2 "" H 5400 3100 50  0000 C CNN
@@
 $EndComp
 $Comp
-L 74LVC14 U12
-U 5 1 58C4719F
-P 5450 3700
-F 0 "U12" H 5600 3800 50  0000 C CNN
-F 1 "74LVC14" H 5650 3600 50  0000 C CNN
-F 2 "SMD_Packages:SOIC-14_N" H 5450 3700 50  0001 C CNN
-F 3 "" H 5450 3700 50  0000 C CNN
-	5    5450 3700
-	1    0    0    -1
-$EndComp
-$Comp
-L GND #PWR59
+L GND #PWR053
 U 1 1 58C471DA
 P 5400 3900
-F 0 "#PWR59" H 5400 3650 50  0001 C CNN
+F 0 "#PWR053" H 5400 3650 50  0001 C CNN
 F 1 "GND" H 5400 3750 50  0000 C CNN
 F 2 "" H 5400 3900 50  0000 C CNN
@@
 $EndComp
 $Comp
-L 74LVC14 U12
-U 6 1 58C4729A
-P 5450 4500
-F 0 "U12" H 5600 4600 50  0000 C CNN
-F 1 "74LVC14" H 5650 4400 50  0000 C CNN
-F 2 "SMD_Packages:SOIC-14_N" H 5450 4500 50  0001 C CNN
-F 3 "" H 5450 4500 50  0000 C CNN
-	6    5450 4500
-	1    0    0    -1
-$EndComp
-$Comp
-L GND #PWR61
+L GND #PWR054
 U 1 1 58C472D8
 P 5400 4700
-F 0 "#PWR61" H 5400 4450 50  0001 C CNN
+F 0 "#PWR054" H 5400 4450 50  0001 C CNN
 F 1 "GND" H 5400 4550 50  0000 C CNN
 F 2 "" H 5400 4700 50  0000 C CNN
@@
 $EndComp
 $Comp
-L GND #PWR49
+L GND #PWR055
 U 1 1 58C4D326
 P 4250 2450
-F 0 "#PWR49" H 4250 2200 50  0001 C CNN
+F 0 "#PWR055" H 4250 2200 50  0001 C CNN
 F 1 "GND" H 4250 2300 50  0000 C CNN
 F 2 "" H 4250 2450 50  0000 C CNN
@@
 divided_clock_in
 $Comp
-L VCC #PWR50
+L VCC #PWR056
 U 1 1 58C5EBC4
 P 4300 1100
-F 0 "#PWR50" H 4300 950 50  0001 C CNN
+F 0 "#PWR056" H 4300 950 50  0001 C CNN
 F 1 "VCC" H 4300 1250 50  0000 C CNN
 F 2 "" H 4300 1100 50  0000 C CNN
@@
 $EndComp
 $Comp
-L VCC #PWR52
+L VCC #PWR057
 U 1 1 58C5EBF1
 P 5400 1100
-F 0 "#PWR52" H 5400 950 50  0001 C CNN
+F 0 "#PWR057" H 5400 950 50  0001 C CNN
 F 1 "VCC" H 5400 1250 50  0000 C CNN
 F 2 "" H 5400 1100 50  0000 C CNN
@@
 $EndComp
 $Comp
-L VCC #PWR54
+L VCC #PWR058
 U 1 1 58C5EC17
 P 5400 1900
-F 0 "#PWR54" H 5400 1750 50  0001 C CNN
+F 0 "#PWR058" H 5400 1750 50  0001 C CNN
 F 1 "VCC" H 5400 2050 50  0000 C CNN
 F 2 "" H 5400 1900 50  0000 C CNN
@@
 $EndComp
 $Comp
-L VCC #PWR56
+L VCC #PWR059
 U 1 1 58C5EC3D
 P 5400 2700
-F 0 "#PWR56" H 5400 2550 50  0001 C CNN
+F 0 "#PWR059" H 5400 2550 50  0001 C CNN
 F 1 "VCC" H 5400 2850 50  0000 C CNN
 F 2 "" H 5400 2700 50  0000 C CNN
@@
 $EndComp
 $Comp
-L VCC #PWR58
+L VCC #PWR060
 U 1 1 58C5EC63
 P 5400 3500
-F 0 "#PWR58" H 5400 3350 50  0001 C CNN
+F 0 "#PWR060" H 5400 3350 50  0001 C CNN
 F 1 "VCC" H 5400 3650 50  0000 C CNN
 F 2 "" H 5400 3500 50  0000 C CNN
@@
 $EndComp
 $Comp
-L VCC #PWR60
+L VCC #PWR061
 U 1 1 58C5EC89
 P 5400 4300
-F 0 "#PWR60" H 5400 4150 50  0001 C CNN
+F 0 "#PWR061" H 5400 4150 50  0001 C CNN
 F 1 "VCC" H 5400 4450 50  0000 C CNN
 F 2 "" H 5400 4300 50  0000 C CNN
@@
 $EndComp
 $Comp
-L VCC #PWR48
+L VCC #PWR062
 U 1 1 58C5EF4C
 P 4250 2150
-F 0 "#PWR48" H 4250 2000 50  0001 C CNN
+F 0 "#PWR062" H 4250 2000 50  0001 C CNN
 F 1 "VCC" H 4250 2300 50  0000 C CNN
 F 2 "" H 4250 2150 50  0000 C CNN
@@
 Text Notes 6100 1050 0    60   ~ 0
 Solder 50ohm resistor from BNC signal pad to BNC signal solder lug
+$Comp
+L 74LVC14 U12
+U 2 1 58D01059
+P 5450 1300
+F 0 "U12" H 5600 1400 50  0000 C CNN
+F 1 "74LVC14" H 5650 1200 50  0000 C CNN
+F 2 "SMD_Packages:SOIC-14_N" H 5450 1300 50  0001 C CNN
+F 3 "http://www.ti.com/lit/ds/symlink/sn74lvc14a.pdf" H 5450 1300 50  0001 C CNN
+F 4 "TI" H 5450 1300 60  0001 C CNN "Manufacturer"
+F 5 "SN74LVC14ADR" H 5450 1300 60  0001 C CNN "Manufacturer PN"
+F 6 "Mouser" H 5450 1300 60  0001 C CNN "Distributor"
+F 7 "595-SN74LVC14ADR" H 5450 1300 60  0001 C CNN "Distributor PN"
+F 8 "http://www.mouser.com/Search/ProductDetail.aspx?R=SN74LVC14ADRvirtualkey59500000virtualkey595-SN74LVC14ADR" H 5450 1300 60  0001 C CNN "URL"
+F 9 "0.40" H 5450 1300 60  0001 C CNN "Unit Price"
+	2    5450 1300
+	1    0    0    -1
+$EndComp
+$Comp
+L 74LVC14 U12
+U 3 1 58D010D3
+P 5450 2100
+F 0 "U12" H 5600 2200 50  0000 C CNN
+F 1 "74LVC14" H 5650 2000 50  0000 C CNN
+F 2 "SMD_Packages:SOIC-14_N" H 5450 2100 50  0001 C CNN
+F 3 "http://www.ti.com/lit/ds/symlink/sn74lvc14a.pdf" H 5450 2100 50  0001 C CNN
+F 4 "TI" H 5450 2100 60  0001 C CNN "Manufacturer"
+F 5 "SN74LVC14ADR" H 5450 2100 60  0001 C CNN "Manufacturer PN"
+F 6 "Mouser" H 5450 2100 60  0001 C CNN "Distributor"
+F 7 "595-SN74LVC14ADR" H 5450 2100 60  0001 C CNN "Distributor PN"
+F 8 "http://www.mouser.com/Search/ProductDetail.aspx?R=SN74LVC14ADRvirtualkey59500000virtualkey595-SN74LVC14ADR" H 5450 2100 60  0001 C CNN "URL"
+F 9 "0.40" H 5450 2100 60  0001 C CNN "Unit Price"
+	3    5450 2100
+	1    0    0    -1
+$EndComp
+$Comp
+L 74LVC14 U12
+U 4 1 58D011BD
+P 5450 2900
+F 0 "U12" H 5600 3000 50  0000 C CNN
+F 1 "74LVC14" H 5650 2800 50  0000 C CNN
+F 2 "SMD_Packages:SOIC-14_N" H 5450 2900 50  0001 C CNN
+F 3 "http://www.ti.com/lit/ds/symlink/sn74lvc14a.pdf" H 5450 2900 50  0001 C CNN
+F 4 "TI" H 5450 2900 60  0001 C CNN "Manufacturer"
+F 5 "SN74LVC14ADR" H 5450 2900 60  0001 C CNN "Manufacturer PN"
+F 6 "Mouser" H 5450 2900 60  0001 C CNN "Distributor"
+F 7 "595-SN74LVC14ADR" H 5450 2900 60  0001 C CNN "Distributor PN"
+F 8 "http://www.mouser.com/Search/ProductDetail.aspx?R=SN74LVC14ADRvirtualkey59500000virtualkey595-SN74LVC14ADR" H 5450 2900 60  0001 C CNN "URL"
+F 9 "0.40" H 5450 2900 60  0001 C CNN "Unit Price"
+	4    5450 2900
+	1    0    0    -1
+$EndComp
+$Comp
+L 74LVC14 U12
+U 5 1 58D0122C
+P 5450 3700
+F 0 "U12" H 5600 3800 50  0000 C CNN
+F 1 "74LVC14" H 5650 3600 50  0000 C CNN
+F 2 "SMD_Packages:SOIC-14_N" H 5450 3700 50  0001 C CNN
+F 3 "http://www.ti.com/lit/ds/symlink/sn74lvc14a.pdf" H 5450 3700 50  0001 C CNN
+F 4 "TI" H 5450 3700 60  0001 C CNN "Manufacturer"
+F 5 "SN74LVC14ADR" H 5450 3700 60  0001 C CNN "Manufacturer PN"
+F 6 "Mouser" H 5450 3700 60  0001 C CNN "Distributor"
+F 7 "595-SN74LVC14ADR" H 5450 3700 60  0001 C CNN "Distributor PN"
+F 8 "http://www.mouser.com/Search/ProductDetail.aspx?R=SN74LVC14ADRvirtualkey59500000virtualkey595-SN74LVC14ADR" H 5450 3700 60  0001 C CNN "URL"
+F 9 "0.40" H 5450 3700 60  0001 C CNN "Unit Price"
+	5    5450 3700
+	1    0    0    -1
+$EndComp
+$Comp
+L 74LVC14 U12
+U 6 1 58D0126B
+P 5450 4500
+F 0 "U12" H 5600 4600 50  0000 C CNN
+F 1 "74LVC14" H 5650 4400 50  0000 C CNN
+F 2 "SMD_Packages:SOIC-14_N" H 5450 4500 50  0001 C CNN
+F 3 "http://www.ti.com/lit/ds/symlink/sn74lvc14a.pdf" H 5450 4500 50  0001 C CNN
+F 4 "TI" H 5450 4500 60  0001 C CNN "Manufacturer"
+F 5 "SN74LVC14ADR" H 5450 4500 60  0001 C CNN "Manufacturer PN"
+F 6 "Mouser" H 5450 4500 60  0001 C CNN "Distributor"
+F 7 "595-SN74LVC14ADR" H 5450 4500 60  0001 C CNN "Distributor PN"
+F 8 "http://www.mouser.com/Search/ProductDetail.aspx?R=SN74LVC14ADRvirtualkey59500000virtualkey595-SN74LVC14ADR" H 5450 4500 60  0001 C CNN "URL"
+F 9 "0.40" H 5450 4500 60  0001 C CNN "Unit Price"
+	6    5450 4500
+	1    0    0    -1
+$EndComp
 $EndSCHEMATC
